File: hw/usb_keyb.sch (KiCad schematic (older format))
At the start: 109 parts, among them J10 SPI, J11 RMII, J12 PS2, J13 OUT_JMP, J14 MTX_JMP, J2 Micro_SD_Card, J3 USB_1, J4 ZX-BUS, J5 MX_ROW, J6 MX_COL, J7 I2C, J8 UART, J9 PROG, SW1 RESET, SW2 OUTPUT, SW3 MATRIX, U1 LM3671MF, U2 STM32F407VETx, U3 STMPS2161STR, U4 NUP4201MR6, U5 74LS245, Y1 8MHz

Commit message: Обновлена плата
Connections:
- net +3V3: no longer R20.1, R21.1, R22.1, R23.1, R24.1, R25.1, R26.1, R27.1, R28.1, R29.1, R30.1, R31.1, R32.1, R33.1, R34.1
- net +5V: now also R20.1, R21.1, R22.1, R23.1, R24.1, R25.1, R26.1, R27.1, R28.1, R29.1, R30.1, R31.1, R32.1, R33.1, R34.1
Changed lines of the file:
@@
 	0    -1   -1   0
-$EndComp
-$Comp
-L +3.3V #PWR010
-U 1 1 5AB14C16
-P 12050 1600
-F 0 "#PWR010" H 12050 1450 50  0001 C CNN
-F 1 "+3.3V" H 12050 1740 50  0000 C CNN
-F 2 "" H 12050 1600 50  0001 C CNN
-F 3 "" H 12050 1600 50  0001 C CNN
-	1    12050 1600
-	1    0    0    -1
 $EndComp
 Text GLabel 8400 1600 0    60   Input ~ 0
@@
 $EndComp
 $Comp
-L +3.3V #PWR029
-U 1 1 5AB415BA
-P 13250 850
-F 0 "#PWR029" H 13250 700 50  0001 C CNN
-F 1 "+3.3V" H 13250 990 50  0000 C CNN
-F 2 "" H 13250 850 50  0001 C CNN
-F 3 "" H 13250 850 50  0001 C CNN
-	1    13250 850
-	1    0    0    -1
-$EndComp
-$Comp
 L R R31
 U 1 1 5AB415C8
@@
 $EndComp
 $Comp
-L +3.3V #PWR030
+L +3.3V #PWR029
 U 1 1 5AB90878
 P 13300 5550
-F 0 "#PWR030" H 13300 5400 50  0001 C CNN
+F 0 "#PWR029" H 13300 5400 50  0001 C CNN
 F 1 "+3.3V" V 13300 5775 50  0000 C CNN
 F 2 "" H 13300 5550 50  0001 C CNN
@@
 $EndComp
 $Comp
-L +3.3V #PWR031
+L +3.3V #PWR030
 U 1 1 5AB90A03
 P 13800 5550
-F 0 "#PWR031" H 13800 5400 50  0001 C CNN
+F 0 "#PWR030" H 13800 5400 50  0001 C CNN
 F 1 "+3.3V" V 13800 5775 50  0000 C CNN
 F 2 "" H 13800 5550 50  0001 C CNN
@@
 $EndComp
 $Comp
-L GND #PWR032
+L GND #PWR031
 U 1 1 5AB90D14
 P 13300 5650
-F 0 "#PWR032" H 13300 5400 50  0001 C CNN
+F 0 "#PWR031" H 13300 5400 50  0001 C CNN
 F 1 "GND" V 13300 5450 50  0000 C CNN
 F 2 "" H 13300 5650 50  0001 C CNN
@@
 $EndComp
 $Comp
-L GND #PWR033
+L GND #PWR032
 U 1 1 5AB91029
 P 13800 5650
-F 0 "#PWR033" H 13800 5400 50  0001 C CNN
+F 0 "#PWR032" H 13800 5400 50  0001 C CNN
 F 1 "GND" V 13800 5450 50  0000 C CNN
 F 2 "" H 13800 5650 50  0001 C CNN
@@
 PS2_DAT
 $Comp
-L +5V #PWR034
+L +5V #PWR033
 U 1 1 5ABBE63D
 P 13800 2550
-F 0 "#PWR034" H 13800 2400 50  0001 C CNN
+F 0 "#PWR033" H 13800 2400 50  0001 C CNN
 F 1 "+5V" V 13800 2725 50  0000 C CNN
 F 2 "" H 13800 2550 50  0001 C CNN
@@
 $EndComp
 $Comp
-L +5V #PWR035
+L +5V #PWR034
 U 1 1 5ABBE907
 P 15600 5550
-F 0 "#PWR035" H 15600 5400 50  0001 C CNN
+F 0 "#PWR034" H 15600 5400 50  0001 C CNN
 F 1 "+5V" V 15600 5725 50  0000 C CNN
 F 2 "" H 15600 5550 50  0001 C CNN
@@
 $EndComp
 $Comp
-L GND #PWR036
+L GND #PWR035
 U 1 1 5ABBEBC0
 P 15600 5450
-F 0 "#PWR036" H 15600 5200 50  0001 C CNN
+F 0 "#PWR035" H 15600 5200 50  0001 C CNN
 F 1 "GND" V 15600 5250 50  0000 C CNN
 F 2 "" H 15600 5450 50  0001 C CNN
@@
 $EndComp
 $Comp
-L GND #PWR037
+L GND #PWR036
 U 1 1 5ABC0107
 P 13800 3650
-F 0 "#PWR037" H 13800 3400 50  0001 C CNN
+F 0 "#PWR036" H 13800 3400 50  0001 C CNN
 F 1 "GND" V 13800 3450 50  0000 C CNN
 F 2 "" H 13800 3650 50  0001 C CNN
@@
 ZD7
 $Comp
-L GND #PWR038
+L GND #PWR037
 U 1 1 5ABE36FB
 P 6200 10100
-F 0 "#PWR038" H 6200 9850 50  0001 C CNN
+F 0 "#PWR037" H 6200 9850 50  0001 C CNN
 F 1 "GND" H 6200 9950 50  0000 C CNN
 F 2 "" H 6200 10100 50  0001 C CNN
@@
 $EndComp
 $Comp
-L +3.3V #PWR039
+L +3.3V #PWR038
 U 1 1 5ABE6543
 P 7200 9350
-F 0 "#PWR039" H 7200 9200 50  0001 C CNN
+F 0 "#PWR038" H 7200 9200 50  0001 C CNN
 F 1 "+3.3V" H 7200 9490 50  0000 C CNN
 F 2 "" H 7200 9350 50  0001 C CNN
@@
 OUT2
 $Comp
-L GND #PWR040
+L GND #PWR039
 U 1 1 5ABEA672
 P 8050 10550
-F 0 "#PWR040" H 8050 10300 50  0001 C CNN
+F 0 "#PWR039" H 8050 10300 50  0001 C CNN
 F 1 "GND" H 8050 10400 50  0000 C CNN
 F 2 "" H 8050 10550 50  0001 C CNN
@@
 $EndComp
 $Comp
-L +3.3V #PWR041
+L +3.3V #PWR040
 U 1 1 5ABEA69C
 P 9500 9350
-F 0 "#PWR041" H 9500 9200 50  0001 C CNN
+F 0 "#PWR040" H 9500 9200 50  0001 C CNN
 F 1 "+3.3V" H 9500 9490 50  0000 C CNN
 F 2 "" H 9500 9350 50  0001 C CNN
@@
 H1_N
 $Comp
-L +3.3V #PWR042
+L +3.3V #PWR041
 U 1 1 5ABE9E17
 P 1750 4150
-F 0 "#PWR042" H 1750 4000 50  0001 C CNN
+F 0 "#PWR041" H 1750 4000 50  0001 C CNN
 F 1 "+3.3V" V 1750 4375 50  0000 C CNN
 F 2 "" H 1750 4150 50  0001 C CNN
@@
 $EndComp
 $Comp
-L GND #PWR043
+L GND #PWR042
 U 1 1 5ABEDD6A
 P 5000 2900
-F 0 "#PWR043" H 5000 2650 50  0001 C CNN
+F 0 "#PWR042" H 5000 2650 50  0001 C CNN
 F 1 "GND" H 5000 2750 50  0000 C CNN
 F 2 "" H 5000 2900 50  0001 C CNN
@@
 $EndComp
 $Comp
-L VCC #PWR044
+L VCC #PWR043
 U 1 1 5AC07BE8
 P 2425 9800
-F 0 "#PWR044" H 2425 9650 50  0001 C CNN
+F 0 "#PWR043" H 2425 9650 50  0001 C CNN
 F 1 "VCC" H 2425 9950 50  0000 C CNN
 F 2 "" H 2425 9800 50  0001 C CNN
@@
 Connection ~ 4350 1050
 $Comp
-L GND #PWR045
+L GND #PWR044
 U 1 1 5AC19DE0
 P 2975 1750
-F 0 "#PWR045" H 2975 1500 50  0001 C CNN
+F 0 "#PWR044" H 2975 1500 50  0001 C CNN
 F 1 "GND" V 2975 1575 50  0000 C CNN
 F 2 "" H 2975 1750 50  0001 C CNN
@@
 $EndComp
 $Comp
-L GND #PWR046
+L GND #PWR045
 U 1 1 5AC325BD
 P 13550 9000
-F 0 "#PWR046" H 13550 8750 50  0001 C CNN
+F 0 "#PWR045" H 13550 8750 50  0001 C CNN
 F 1 "GND" H 13550 8850 50  0000 C CNN
 F 2 "" H 13550 9000 50  0001 C CNN
@@
 	13400 8550 13550 8550
 Connection ~ 13550 8750
+$Comp
+L +5V #PWR046
+U 1 1 5AC80AD3
+P 13250 850
+F 0 "#PWR046" H 13250 700 50  0001 C CNN
+F 1 "+5V" H 13250 1000 50  0000 C CNN
+F 2 "" H 13250 850 50  0001 C CNN
+F 3 "" H 13250 850 50  0001 C CNN
+	1    13250 850
+	1    0    0    -1
+$EndComp
+$Comp
+L +5V #PWR?
+U 1 1 5AC81741
+P 12050 1600
+F 0 "#PWR?" H 12050 1450 50  0001 C CNN
+F 1 "+5V" H 12050 1750 50  0000 C CNN
+F 2 "" H 12050 1600 50  0001 C CNN
+F 3 "" H 12050 1600 50  0001 C CNN
+	1    12050 1600
+	1    0    0    -1
+$EndComp
 $EndSCHEMATC
